File: Hardware/YF-SA600H/btn.kicad_sch (KiCad schematic)
At the start: 2 parts

Commit message: Add buttons
Other:
- title: YardForce SA600H LCD CoverUI HS49067 -> YardForce SAxxxPRO Dot-Matrix LCD CoverUI HS49067
Changed lines of the file:
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@@
   (paper "A4")
   (title_block
-    (title "YardForce SA600H LCD CoverUI HS49067")
+    (title "YardForce SAxxxPRO Dot-Matrix LCD CoverUI HS49067")
     (date "2023-08-22")
     (rev "0.1")
