File: Hardware/YF-SA600H/mcu_stm32f030.kicad_sch (KiCad schematic)
At the start: 9 parts, among them U3 STM32F030RCTx

Commit message: Add buttons
Other:
- title: YardForce SA600H LCD CoverUI HS49067 -> YardForce SAxxxPRO Dot-Matrix LCD CoverUI HS49067
Changed lines of the file:
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@@
   (paper "A4")
   (title_block
-    (title "YardForce SA600H LCD CoverUI HS49067")
+    (title "YardForce SAxxxPRO Dot-Matrix LCD CoverUI HS49067")
     (date "2023-08-22")
     (rev "0.1")
@@
     (effects (font (size 1.27 1.27)) (justify right bottom))
   )
-  (label "U2.PB15" (at 156.21 129.54 0)
+  (label "U3.PB15" (at 156.21 129.54 0)
     (effects (font (size 1.27 1.27)) (justify left bottom))
   )
@@
     (effects (font (size 1.27 1.27)) (justify left bottom))
   )
-  (label "U2.PC1" (at 93.98 93.98 0)
+  (label "U3.PC1" (at 93.98 93.98 0)
     (effects (font (size 1.27 1.27)) (justify left bottom))
   )
@@
     (effects (font (size 1.27 1.27)) (justify left bottom))
   )
-  (label "U2.PC3" (at 93.98 99.06 0)
+  (label "U3.PC3" (at 93.98 99.06 0)
     (effects (font (size 1.27 1.27)) (justify left bottom))
   )
@@
     (effects (font (size 1.27 1.27)) (justify left bottom))
   )
-  (label "U2.PC0" (at 93.98 91.44 0)
+  (label "U3.PC0" (at 93.98 91.44 0)
     (effects (font (size 1.27 1.27)) (justify left bottom))
   )
@@
     (effects (font (size 1.27 1.27)) (justify left bottom))
   )
-  (label "U2.PB12" (at 156.21 121.92 0)
-    (effects (font (size 1.27 1.27)) (justify left bottom))
-  )
+  (label "U3.PB12" (at 156.21 121.92 0)
+    (effects (font (size 1.27 1.27)) (justify left bottom))
+  )
