File: Hardware/YardForce/Subsheets/NX100i 18Button-3LED-LCD Board/btns-leds-lcd.kicad_sch (KiCad schematic)
At the start: 34 parts, among them Q1 Q_NPN_BEC

Commit message: NX100i general done
Other:
- note added: "A0(RS), DATA/~{CMD}"
- note added: "E(RD)"
- note added: "Model: JLX25664G-251-BN Matrix: 256*64 Pixel Outer Dim: 67mm * 30mm Driver: ST75256"
- note added: "RW(WR)"
- note removed: "A0/RS, DATA/~{CMD}"
- note removed: "Model : JLX12832A-3G Cable : JLX256128G - 256 Matrix: 128*32 Pixel Driver: ST75256"
- note removed: "RD"
- note removed: "WR"
Changed lines of the file:
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@@
     (stroke (width 0) (type default) (color 0 0 0 0))
   )
-  (text "WR" (at 96.52 68.58 90)
+  (text "RW(WR)" (at 96.52 68.58 90)
     (effects (font (size 1.27 1.27)) (justify left bottom))
   )
@@
     (effects (font (size 1.27 1.27)) (justify left bottom))
   )
-  (text "Model : JLX12832A-3G\nCable : JLX256128G - 256\nMatrix: 128*32 Pixel\nDriver: ST75256"
-    (at 71.12 49.53 0)
+  (text "Model: JLX25664G-251-BN\nMatrix: 256*64 Pixel\nOuter Dim: 67mm * 30mm\nDriver: ST75256"
+    (at 67.31 49.53 0)
     (effects (font (size 2 2)) (justify left bottom))
   )
@@
     (effects (font (size 1.27 1.27)) (justify left bottom))
   )
-  (text "RD" (at 93.98 68.58 90)
+  (text "E(RD)" (at 93.98 68.58 90)
     (effects (font (size 1.27 1.27)) (justify left bottom))
   )
@@
     (effects (font (size 1.27 1.27)) (justify left bottom))
   )
-  (text "A0/RS, DATA/~{CMD}" (at 91.44 68.58 90)
+  (text "A0(RS), DATA/~{CMD}" (at 91.44 68.58 90)
     (effects (font (size 1.27 1.27)) (justify left bottom))
   )
