File: Hardware/YardForce/NX100i 18Button-3LED-LCD Board.kicad_sch (KiCad schematic)
At the start: 15 parts, among them U1 AMS1117 3.3 2028

Commit message: Final cosmetic changes
Other:
- note removed: "Optional (MOD_HALL): Solder Cable fro R61/Q4 to U5/Pin-3 to get Signal to PB7"
- note removed: "Optional (MOD_HALL): Solder Cable from R74/Q5 to U5 (Pin 2) to get Stop Hall (ST2) to GPIO PB6"
- note removed: "Optional (MOD_HALL): Solder Cable from R83/Q6 to U5/Pin-10 to get Signal to PB8"
