File: Hardware/YardForce/SA,SC-Type 10Button-12LED Board.kicad_sch (KiCad schematic)
At the start: 22 parts, among them U3 AMS1117-3.3

Commit message: Add MOD_HALL to RM-ECOW-V1.0.0
Parts:
- renumbered JP2 to JP7
