File: Hardware/YardForce/Subsheets/SA,SC-Type 10Button-12LED Board/mcu_stm32f030.kicad_sch (KiCad schematic)
At the start: 3 parts, among them U1 STM32F030R8Tx, U2 ESP-WROOM-02

Commit message: Evaluated Hall Support
Parts:
- added R33: 4k7, symbol Device:R
Connections:
- net GND: now also R33.1
- net at U1.60 (BOOT0): now also R33.2
Changed lines of the file:
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@@
+    (stroke (width 0) (type default) (color 0 0 0 0))
+  )
+  (wire (pts (xy 96.52 55.88) (xy 96.52 53.34))
     (stroke (width 0) (type default) (color 0 0 0 0))
   )
@@
     (stroke (width 0) (type default) (color 0 0 0 0))
   )
+  (wire (pts (xy 106.68 53.34) (xy 111.76 53.34))
+    (stroke (width 0) (type default) (color 0 0 0 0))
+  )
   (bus (pts (xy 167.64 106.68) (xy 167.64 109.22))
+    (stroke (width 0) (type default) (color 0 0 0 0))
+  )
+  (wire (pts (xy 96.52 53.34) (xy 99.06 53.34))
     (stroke (width 0) (type default) (color 0 0 0 0))
   )
@@
     (pin "9")
   )
+  (symbol (lib_id "Device:R") (at 102.87 53.34 90) (unit 1)
+    (in_bom yes) (on_board yes)
+    (property "Reference" "R33" (id 0) (at 102.87 53.34 90))
+    (property "Value" "4k7" (id 1) (at 105.41 55.88 90))
+    (property "Footprint" "" (id 2) (at 102.87 55.118 90)
+      (effects (font (size 1.27 1.27)) hide)
+    )
+    (property "Datasheet" "~" (id 3) (at 102.87 53.34 0)
+      (effects (font (size 1.27 1.27)) hide)
+    )
+    (pin "1")
+    (pin "2")
+  )
+  (symbol (lib_id "power:GND") (at 96.52 55.88 0) (unit 1)
+    (in_bom yes) (on_board yes)
+    (property "Reference" "#PWR?" (id 0) (at 96.52 62.23 0)
+      (effects (font (size 1.27 1.27)) hide)
+    )
+    (property "Value" "GND" (id 1) (at 96.647 60.2742 0))
+    (property "Footprint" "" (id 2) (at 96.52 55.88 0)
+      (effects (font (size 1.27 1.27)) hide)
+    )
+    (property "Datasheet" "" (id 3) (at 96.52 55.88 0)
+      (effects (font (size 1.27 1.27)) hide)
+    )
+    (pin "1")
+  )
   (symbol (lib_id "power:+3.3V") (at 218.44 64.77 0) (unit 1)

Commit message: Add MOD_HALL to RM-ECOW-V1.0.0
Parts:
- added C1: C, symbol Device:C
- added R34: NP, symbol Device:R
- R37: now not fitted
Connections:
- net GND: now also U2.5 (IO13), C1.2
- net at U1.13 (VDDA): now also R34.2
- net at U1.7 (NRST): now also C1.1, R34.1
- no-connect marks 0 -> 21
Other:
- note added: "Optional (MOD_HALL): Solder 4 Cables: 1. JP2 Pin10 to U2 Pin6 (to get LIFTX on PF6) 2. JP2 Pin12 to U2 Pin7 (to get LBUMP on PA12) 3. JP2 Pin15 to U2 Pin8 (to get RBUMP on PA11) 4. JP2 Pin16 to U2 Pin17 (to get LIFT on PA8)"
